File: Hardware/SparkFun_LilyPad_Main_Board.sch (EAGLE design)
At the start: 39 parts, among them U1 ATMEGA328P_TQFP, Y1 8MHZ

Commit message: Updates for QC checklist
Parts:
- added FID1, FID2: FIDUCIALUFIDUCIAL, SparkFun-Aesthetics:FIDUCIALUFIDUCIAL
Other:
- note added: "Operational voltage 2.7-5.5v Compatible with 3.3 or 5v FTDI (Lilypad FTDI is 5v) *DISCONNECT BATTERY BEFORE PLUGGING IN FTDI BOARD*"
Changed lines of the file:
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@@
 <setting verticaltext="up"/>
 </settings>
-<grid distance="0.1" unitdist="inch" unit="inch" style="lines" multiple="1" display="no" altdistance="0.01" altunitdist="inch" altunit="inch"/>
+<grid distance="0.05" unitdist="inch" unit="inch" style="lines" multiple="1" display="yes" altdistance="0.005" altunitdist="inch" altunit="inch"/>
 <layers>
 <layer number="1" name="Top" color="4" fill="1" visible="no" active="no"/>
@@
 <part name="S1" library="SparkFun-Electromechanical" deviceset="SWITCH-MOMENTARY-2" device="SMD-REDUNDANT"/>
 <part name="U$22" library="SparkFun-Aesthetics" deviceset="REVISION" device=""/>
+<part name="FID1" library="SparkFun-Aesthetics" deviceset="FIDUCIAL" device="UFIDUCIAL"/>
+<part name="FID2" library="SparkFun-Aesthetics" deviceset="FIDUCIAL" device="UFIDUCIAL"/>
+<part name="GND10" library="SparkFun-Aesthetics" deviceset="GND" device=""/>
+<part name="P+8" library="SparkFun-Aesthetics" deviceset="VCC" device=""/>
 </parts>
 <sheets>
@@
 <text x="170.942" y="6.858" size="2.1844" layer="94" font="vector">Dia Campbell</text>
 <text x="238.76" y="7.62" size="2.1844" layer="94" font="vector">v21</text>
+<text x="175.26" y="170.18" size="1.778" layer="91">Operational voltage 2.7-5.5v
+Compatible with 3.3 or 5v FTDI
+(Lilypad FTDI is 5v)
+*DISCONNECT BATTERY BEFORE PLUGGING IN FTDI BOARD*</text>
 </plain>
 <instances>
@@
 <instance part="FRAME1" gate="V" x="147.32" y="0"/>
 <instance part="U1" gate="U$1" x="127" y="116.84" smashed="yes">
-<attribute name="NAME" x="109.22" y="145.288" size="1.778" layer="95"/>
-<attribute name="VALUE" x="109.474" y="78.486" size="1.778" layer="96"/>
+<attribute name="NAME" x="114.3" y="150.368" size="1.778" layer="95"/>
+<attribute name="VALUE" x="113.03" y="82.296" size="1.778" layer="96"/>
 </instance>
 <instance part="U$2" gate="G$1" x="172.72" y="144.78" smashed="yes"/>
@@
 <instance part="U$1" gate="G$1" x="172.72" y="147.32" smashed="yes"/>
 <instance part="$0000003" gate="G$1" x="236.22" y="17.78"/>
-<instance part="JP3" gate="G$1" x="43.18" y="43.18"/>
+<instance part="JP3" gate="G$1" x="43.18" y="43.18" smashed="yes">
+<attribute name="NAME" x="38.862" y="49.022" size="1.778" layer="95"/>
+</instance>
 <instance part="P+1" gate="G$1" x="63.5" y="48.26" smashed="yes">
 <attribute name="VALUE" x="62.484" y="51.816" size="1.778" layer="96"/>
@@
 </instance>
 <instance part="U$22" gate="G$1" x="149.098" y="6.858"/>
+<instance part="FID1" gate="G$1" x="200.66" y="33.02"/>
+<instance part="FID2" gate="G$1" x="205.74" y="33.02"/>
+<instance part="GND10" gate="1" x="104.14" y="45.72"/>
+<instance part="P+8" gate="G$1" x="93.98" y="60.96" smashed="yes">
+<attribute name="VALUE" x="92.964" y="58.674" size="1.778" layer="96" rot="R90"/>
+</instance>
 </instances>
 <busses>
@@
 <wire x1="111.76" y1="55.88" x2="104.14" y2="55.88" width="0.1524" layer="91"/>
 <pinref part="JP1" gate="G$1" pin="CTS"/>
-<label x="104.14" y="55.88" size="1.27" layer="95" font="vector" rot="R180" xref="yes"/>
-</segment>
-<segment>
+<pinref part="GND10" gate="1" pin="GND"/>
+<wire x1="104.14" y1="55.88" x2="104.14" y2="53.34" width="0.1524" layer="91"/>
+<wire x1="104.14" y1="53.34" x2="104.14" y2="48.26" width="0.1524" layer="91"/>
 <wire x1="111.76" y1="53.34" x2="104.14" y2="53.34" width="0.1524" layer="91"/>
 <pinref part="JP1" gate="G$1" pin="GND"/>
-<label x="104.14" y="53.34" size="1.27" layer="95" font="vector" rot="R180" xref="yes"/>
+<junction x="104.14" y="53.34"/>
 </segment>
 <segment>
@@
 </segment>
 <segment>
-<wire x1="111.76" y1="58.42" x2="104.14" y2="58.42" width="0.1524" layer="91"/>
 <pinref part="JP1" gate="G$1" pin="VCC"/>
-<label x="104.14" y="58.42" size="1.27" layer="95" font="vector" rot="R180" xref="yes"/>
+<pinref part="P+8" gate="G$1" pin="VCC"/>
+<wire x1="111.76" y1="58.42" x2="93.98" y2="58.42" width="0.1524" layer="91"/>
+<wire x1="93.98" y1="58.42" x2="93.98" y2="60.96" width="0.1524" layer="91"/>
 </segment>
 <segment>
@@
 </schematic>
 </drawing>
+<compatibility>
+<note version="6.3" minversion="6.2.2" severity="warning">
+Since Version 6.2.2 text objects can contain more than one line,
+which will not be processed correctly with this version.
+</note>
+</compatibility>
 </eagle>

Commit message: Moving logos to bottom copper, removed some silk
Parts:
- JP3: device SparkFun-Connectors:AVR_SPI_PRG_6PTH -> SparkFun-Connectors:AVR_SPI_PRG_6NS
- LOGO1: value SFE_LOGO_FLAME.3_INCH -> SFE_LOGO_FLAME.3COP; device SparkFun-Aesthetics:SFE_LOGO_FLAME.3_INCH -> SparkFun-Aesthetics:SFE_LOGO_FLAME.3COP
- LOGO2: value OSHW-LOGOL -> OSHW-LOGO-COPPERM; device SparkFun-Aesthetics:OSHW-LOGOL -> SparkFun-Aesthetics:OSHW-LOGO-COPPERM
Changed lines of the file:
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@@
 <setting verticaltext="up"/>
 </settings>
-<grid distance="0.05" unitdist="inch" unit="inch" style="lines" multiple="1" display="yes" altdistance="0.005" altunitdist="inch" altunit="inch"/>
+<grid distance="0.1" unitdist="inch" unit="inch" style="lines" multiple="1" display="no" altdistance="0.01" altunitdist="inch" altunit="inch"/>
 <layers>
 <layer number="1" name="Top" color="4" fill="1" visible="no" active="no"/>
@@
 <part name="U$1" library="LilyPad-Wearables" deviceset="SEWTAP" device="9"/>
 <part name="$0000003" library="LilyPad-Wearables" deviceset="LOGO-LP" device="LPA"/>
-<part name="JP3" library="SparkFun-Connectors" deviceset="AVR_SPI_PRG_6" device="PTH" value="FEMALE 2x3"/>
+<part name="JP3" library="SparkFun-Connectors" deviceset="AVR_SPI_PRG_6" device="NS" value="FEMALE 2x3"/>
 <part name="P+1" library="SparkFun-Aesthetics" deviceset="VCC" device=""/>
 <part name="GND1" library="SparkFun-Aesthetics" deviceset="GND" device=""/>
@@
 <part name="JP1" library="SparkFun-Connectors" deviceset="ARDUINO_SERIAL_PROGRAM" device="SMD"/>
 <part name="C1" library="SparkFun-Capacitors" deviceset="0.1UF-25V(+80/-20%)(0603)" device="" value="0.1uF"/>
-<part name="LOGO1" library="SparkFun-Aesthetics" deviceset="SFE_LOGO_FLAME" device=".3_INCH"/>
-<part name="LOGO2" library="SparkFun-Aesthetics" deviceset="OSHW-LOGO" device="L"/>
+<part name="LOGO1" library="SparkFun-Aesthetics" deviceset="SFE_LOGO_FLAME" device=".3COP" value="SFE_LOGO_FLAME.3COP"/>
+<part name="LOGO2" library="SparkFun-Aesthetics" deviceset="OSHW-LOGO-COPPER" device="M"/>
 <part name="S1" library="SparkFun-Electromechanical" deviceset="SWITCH-MOMENTARY-2" device="SMD-REDUNDANT"/>
 <part name="U$22" library="SparkFun-Aesthetics" deviceset="REVISION" device=""/>

Commit message: Made pin 13 LED blue; current standard
Parts:
- D1: value GREEN -> BLUE; device SparkFun-LED:LED-GREEN0603 -> SparkFun-LED:LED-BLUE0603
Changed lines of the file:
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@@
 <part name="U$7" library="LilyPad-Wearables" deviceset="SEWTAP" device="9"/>
 <part name="U$14" library="LilyPad-Wearables" deviceset="SEWTAP" device="9"/>
-<part name="D1" library="SparkFun-LED" deviceset="LED-GREEN" device="0603" value="GREEN"/>
+<part name="D1" library="SparkFun-LED" deviceset="LED-BLUE" device="0603" value="BLUE"/>
 <part name="R2" library="SparkFun-Resistors" deviceset="330OHM1/10W1%(0603)" device="" value="330"/>
 <part name="GND2" library="SparkFun-Aesthetics" deviceset="GND" device=""/>
